Commit message: Reset dynamixel_node to a placeholder DynamixelServos plugin
Port and baud rate move out of the ros2_control config to the plugin;
per-joint `id` becomes `servo_id`; both launch files default to
dynamixel_node/DynamixelServos, and servo_sim switches mock/real from two
constants at the top. Drops the velocity bridges, which keyboard_control.py
already replaces.

Co-Authored-By: Claude Opus 5 <noreply@anthropic.com>

File: src/arm_moveit_config/config/arm.ros2_control.xacro (robot description, xacro)
@@ -1,23 +1,18 @@
 <?xml version="1.0"?>
 <robot xmlns:xacro="http://www.ros.org/wiki/xacro">
-    <xacro:macro name="arm_ros2_control" params="name initial_positions_file use_mock_hardware:=false hardware_plugin:=mock_components/GenericSystem port:=/dev/ttyUSB0 baud_rate:=1000000">
+    <xacro:macro name="arm_ros2_control" params="name initial_positions_file use_mock_hardware:=false hardware_plugin:=dynamixel_node/DynamixelServos">
         <xacro:property name="initial_positions" value="${xacro.load_yaml(initial_positions_file)['initial_positions']}"/>
         <ros2_control name="${name}" type="system">
             <hardware>
-                <!--
-                     use_mock_hardware:=true for simulation, or point the
-                     hardware_plugin at your own servo hardware_interface plugin.
-                     use_mock_hardware:=false  -->
                 <xacro:if value="${use_mock_hardware}">
                   <plugin>mock_components/GenericSystem</plugin>
                 </xacro:if>
                 <xacro:unless value="${use_mock_hardware}">
+                  <!-- Port and baud rate are owned by the hardware plugin, not this config. -->
                   <plugin>${hardware_plugin}</plugin>
-                  <param name="port">${port}</param>
-                  <param name="baud_rate">${baud_rate}</param>
                 </xacro:unless>
             </hardware>
             <joint name="shoulder_tilt">
-                <param name="id">2</param>
+                <param name="servo_id">2</param>
                 <command_interface name="position"/>
                 <state_interface name="position">
@@ -27,5 +22,5 @@
             </joint>
             <joint name="shoulder_pan">
-                <param name="id">1</param>
+                <param name="servo_id">1</param>
                 <command_interface name="position"/>
                 <state_interface name="position">
@@ -35,5 +30,5 @@
             </joint>
             <joint name="elbow">
-                <param name="id">3</param>
+                <param name="servo_id">3</param>
                 <command_interface name="position"/>
                 <state_interface name="position">
@@ -43,5 +38,5 @@
             </joint>
             <joint name="wrist_pitch">
-                <param name="id">4</param>
+                <param name="servo_id">4</param>
                 <command_interface name="position"/>
                 <state_interface name="position">
@@ -51,5 +46,5 @@
             </joint>
             <joint name="wrist_roll">
-                <param name="id">5</param>
+                <param name="servo_id">5</param>
                 <command_interface name="position"/>
                 <state_interface name="position">
@@ -58,7 +53,8 @@
                 <state_interface name="velocity"/>
             </joint>
+            <!-- TODO: prismatic joint in metres driven by a rotary servo; needs a conversion. -->
             <!-- right_finger_joint is a URDF mimic; ros2_control mirrors it. -->
             <joint name="left_finger_joint">
-                <param name="id">6</param>
+                <param name="servo_id">6</param>
                 <command_interface name="position"/>
                 <state_interface name="position">
@@ -67,4 +63,5 @@
                 <state_interface name="velocity"/>
             </joint>
+            <!-- Gearbox reductions. The hardware plugin must apply these; ros2_control only parses them. -->
             <transmission name="shoulder_pan_drive">
                 <plugin>transmission_interface/SimpleTransmission</plugin>
@@ -97,4 +94,5 @@
                 </actuator>
             </transmission>
+            <!-- Servos 4 and 5 jointly drive pitch and roll. -->
             <transmission name="wrist_differential">
                 <plugin>transmission_interface/DifferentialTransmission</plugin>

File: src/arm_moveit_config/config/arm.urdf.xacro (robot description, xacro)
@@ -3,11 +3,9 @@
     <xacro:arg name="initial_positions_file" default="initial_positions.yaml" />
     <xacro:arg name="use_mock_hardware" default="true" />
-    <xacro:arg name="hardware_plugin" default="mock_components/GenericSystem" />
-    <xacro:arg name="port" default="/dev/ttyUSB0" />
-    <xacro:arg name="baud_rate" default="1000000" />
+    <xacro:arg name="hardware_plugin" default="dynamixel_node/DynamixelServos" />
     <!-- Import arm urdf file -->
     <xacro:include filename="$(find arm_moveit_config)/src/moveit/arm.urdf" />
     <!-- Import control_xacro -->
     <xacro:include filename="arm.ros2_control.xacro" />
-    <xacro:arm_ros2_control name="DynamixelServos" initial_positions_file="$(arg initial_positions_file)" use_mock_hardware="$(arg use_mock_hardware)" hardware_plugin="$(arg hardware_plugin)" port="$(arg port)" baud_rate="$(arg baud_rate)"/>
+    <xacro:arm_ros2_control name="DynamixelServos" initial_positions_file="$(arg initial_positions_file)" use_mock_hardware="$(arg use_mock_hardware)" hardware_plugin="$(arg hardware_plugin)"/>
 </robot>
