Commit message: Add gripper and wrist velocity bridges, enhance keyboard control, and update URDF
- Introduced `gripper_velocity_bridge.py` to convert gripper velocity commands into position targets for the gripper's trajectory controller.
- Added `wrist_velocity_bridge.py` to handle wrist bend and twist velocity commands, integrating them into the wrist trajectory controller.
- Enhanced `keyboard_control.py` to support gripper commands (open, close, and step) and adjust speeds dynamically.
- Created `patch_moveit_servo.sh` for vendoring a patched version of MoveIt Servo.
- Added `urdf_to_openrave.py` for converting URDF to OpenRAVE XML format, focusing on the arm's kinematic chain.
- Updated the arm's URDF to include a parallel-jaw gripper with prismatic joints for each finger, improving the model's fidelity.

File: src/arm_moveit_config/config/arm.ros2_control.xacro (robot description, xacro)
@@ -55,9 +55,10 @@
                 <state_interface name="velocity"/>
             </joint>
-            <joint name="fake_dof">
+            <!-- right_finger_joint is a URDF mimic; ros2_control mirrors it. -->
+            <joint name="left_finger_joint">
                 <command_interface name="position"/>
                 <command_interface name="velocity"/>
                 <state_interface name="position">
-                  <param name="initial_value">${initial_positions['fake_dof']}</param>
+                  <param name="initial_value">${initial_positions['left_finger_joint']}</param>
                 </state_interface>
                 <state_interface name="velocity"/>

File: src/arm_moveit_config/src/moveit/arm.urdf (robot description, URDF)
Before this commit: robot arm, 9 links, 8 joints
Links:
- removed link end_effector
- removed link fake_dof_link
- added link grasp_link
- added link gripper_base, mass 0.05; collision box size=0.035 0.035 0.022; visual box size=0.035 0.035 0.022
- added link left_finger, mass 0.012; collision box size=0.01 0.008 0.04; visual box size=0.01 0.008 0.04
- added link right_finger, mass 0.012; collision box size=0.01 0.008 0.04; visual box size=0.01 0.008 0.04
- link forearm_tip: geometry visual sphere radius=0.01
- link wrist_pitch_link: geometry collision box size=0.04 0.05 0.028; visual box size=0.04 0.05 0.028
- link wrist_roll_link: mass 0.15 -> 0.05; geometry collision box size=0.035 0.035 0.006; visual box size=0.035 0.035 0.006
Joints:
- removed joint end_effector_mount
- removed joint fake_dof
- added joint grasp_frame: type fixed, parent gripper_base, child grasp_link, origin xyz=0 0 0.045 rpy=0 0 0
- added joint gripper_mount: type fixed, parent wrist_roll_link, child gripper_base, origin xyz=0 0 0.006 rpy=0 0 0
- added joint left_finger_joint: type prismatic, parent gripper_base, child left_finger, origin xyz=0 0.004 0.022 rpy=0 0 0, axis 0 1 0, limit lower=0.0 upper=0.015 effort=20.0 velocity=0.1
- added joint right_finger_joint: type prismatic, parent gripper_base, child right_finger, origin xyz=0 -0.004 0.022 rpy=0 0 0, axis 0 -1 0, limit lower=0.0 upper=0.015 effort=20.0 velocity=0.1, mimic joint=left_finger_joint multiplier=1.0 offset=0.0
- joint wrist_roll: limit lower=-3.14159 upper=3.14159 effort=10.0 velocity=2.0 -> lower=-6.28318 upper=6.28318 effort=10.0 velocity=2.0; origin xyz=0 0 0.04 rpy=0 0 0 -> xyz=0 0 0.028 rpy=0 0 0

Commit message: Refactor Dynamixel Node for ros2_control Integration
- Removed the standalone launch file for the Dynamixel node.
- Updated package.xml to reflect changes in dependencies and description.
- Introduced DynamixelController class to handle servo operations and communication.
- Replaced the previous DynamixelNode implementation with a new system interface for ros2_control.
- Implemented DynamixelSystem class to manage multiple servos and their states.
- Added diagnostics publishing for monitoring servo status and bus health.
- Enhanced error handling and logging throughout the codebase.

File: src/arm_moveit_config/config/arm.ros2_control.xacro (robot description, xacro)
@@ -1,11 +1,12 @@
 <?xml version="1.0"?>
 <robot xmlns:xacro="http://www.ros.org/wiki/xacro">
-    <xacro:macro name="arm_ros2_control" params="name initial_positions_file use_mock_hardware:=false hardware_plugin:=mock_components/GenericSystem">
+    <xacro:macro name="arm_ros2_control" params="name initial_positions_file use_mock_hardware:=false hardware_plugin:=mock_components/GenericSystem port:=/dev/ttyUSB0 baud_rate:=1000000">
         <xacro:property name="initial_positions" value="${xacro.load_yaml(initial_positions_file)['initial_positions']}"/>
         <ros2_control name="${name}" type="system">
             <hardware>
-                <!-- This package ships no hardware driver of its own. Leave
-                     use_mock_hardware:=true for simulation, or point
-                     hardware_plugin at your own servo hardware_interface plugin. -->
+                <!--
+                     use_mock_hardware:=true for simulation, or point the
+                     hardware_plugin at your own servo hardware_interface plugin.
+                     use_mock_hardware:=false  -->
                 <xacro:if value="${use_mock_hardware}">
                   <plugin>mock_components/GenericSystem</plugin>
@@ -13,9 +14,11 @@
                 <xacro:unless value="${use_mock_hardware}">
                   <plugin>${hardware_plugin}</plugin>
+                  <param name="port">${port}</param>
+                  <param name="baud_rate">${baud_rate}</param>
                 </xacro:unless>
             </hardware>
             <joint name="shoulder_tilt">
+                <param name="id">2</param>
                 <command_interface name="position"/>
-                <command_interface name="velocity"/>
                 <state_interface name="position">
                   <param name="initial_value">${initial_positions['shoulder_tilt']}</param>
@@ -24,6 +27,6 @@
             </joint>
             <joint name="shoulder_pan">
+                <param name="id">1</param>
                 <command_interface name="position"/>
-                <command_interface name="velocity"/>
                 <state_interface name="position">
                   <param name="initial_value">${initial_positions['shoulder_pan']}</param>
@@ -32,6 +35,6 @@
             </joint>
             <joint name="elbow">
+                <param name="id">3</param>
                 <command_interface name="position"/>
-                <command_interface name="velocity"/>
                 <state_interface name="position">
                   <param name="initial_value">${initial_positions['elbow']}</param>
@@ -40,6 +43,6 @@
             </joint>
             <joint name="wrist_pitch">
+                <param name="id">4</param>
                 <command_interface name="position"/>
-                <command_interface name="velocity"/>
                 <state_interface name="position">
                   <param name="initial_value">${initial_positions['wrist_pitch']}</param>
@@ -48,6 +51,6 @@
             </joint>
             <joint name="wrist_roll">
+                <param name="id">5</param>
                 <command_interface name="position"/>
-                <command_interface name="velocity"/>
                 <state_interface name="position">
                   <param name="initial_value">${initial_positions['wrist_roll']}</param>
@@ -57,6 +60,6 @@
             <!-- right_finger_joint is a URDF mimic; ros2_control mirrors it. -->
             <joint name="left_finger_joint">
+                <param name="id">6</param>
                 <command_interface name="position"/>
-                <command_interface name="velocity"/>
                 <state_interface name="position">
                   <param name="initial_value">${initial_positions['left_finger_joint']}</param>
@@ -64,4 +67,51 @@
                 <state_interface name="velocity"/>
             </joint>
+            <transmission name="shoulder_pan_drive">
+                <plugin>transmission_interface/SimpleTransmission</plugin>
+                <joint name="shoulder_pan" role="joint1">
+                    <mechanical_reduction>1.0</mechanical_reduction>
+                    <offset>0.0</offset>
+                </joint>
+                <actuator name="shoulder_pan_servo" role="actuator1">
+                    <mechanical_reduction>1.0</mechanical_reduction>
+                </actuator>
+            </transmission>
+            <transmission name="shoulder_tilt_drive">
+                <plugin>transmission_interface/SimpleTransmission</plugin>
+                <joint name="shoulder_tilt" role="joint1">
+                    <mechanical_reduction>1.0</mechanical_reduction>
+                    <offset>0.0</offset>
+                </joint>
+                <actuator name="shoulder_tilt_servo" role="actuator1">
+                    <mechanical_reduction>1.0</mechanical_reduction>
+                </actuator>
+            </transmission>
+            <transmission name="elbow_drive">
+                <plugin>transmission_interface/SimpleTransmission</plugin>
+                <joint name="elbow" role="joint1">
+                    <mechanical_reduction>1.0</mechanical_reduction>
+                    <offset>0.0</offset>
+                </joint>
+                <actuator name="elbow_servo" role="actuator1">
+                    <mechanical_reduction>1.0</mechanical_reduction>
+                </actuator>
+            </transmission>
+            <transmission name="wrist_differential">
+                <plugin>transmission_interface/DifferentialTransmission</plugin>
+                <joint name="wrist_pitch" role="joint1">
+                    <mechanical_reduction>1.0</mechanical_reduction>
+                    <offset>0.0</offset>
+                </joint>
+                <joint name="wrist_roll" role="joint2">
+                    <mechanical_reduction>1.0</mechanical_reduction>
+                    <offset>0.0</offset>
+                </joint>
+                <actuator name="wrist_servo_a" role="actuator1">
+                    <mechanical_reduction>1.0</mechanical_reduction>
+                </actuator>
+                <actuator name="wrist_servo_b" role="actuator2">
+                    <mechanical_reduction>1.0</mechanical_reduction>
+                </actuator>
+            </transmission>
         </ros2_control>
     </xacro:macro>

File: src/arm_moveit_config/config/arm.urdf.xacro (robot description, xacro)
@@ -4,8 +4,10 @@
     <xacro:arg name="use_mock_hardware" default="true" />
     <xacro:arg name="hardware_plugin" default="mock_components/GenericSystem" />
+    <xacro:arg name="port" default="/dev/ttyUSB0" />
+    <xacro:arg name="baud_rate" default="1000000" />
     <!-- Import arm urdf file -->
     <xacro:include filename="$(find arm_moveit_config)/src/moveit/arm.urdf" />
     <!-- Import control_xacro -->
     <xacro:include filename="arm.ros2_control.xacro" />
-    <xacro:arm_ros2_control name="FakeSystem" initial_positions_file="$(arg initial_positions_file)" use_mock_hardware="$(arg use_mock_hardware)" hardware_plugin="$(arg hardware_plugin)"/>
+    <xacro:arm_ros2_control name="DynamixelServos" initial_positions_file="$(arg initial_positions_file)" use_mock_hardware="$(arg use_mock_hardware)" hardware_plugin="$(arg hardware_plugin)" port="$(arg port)" baud_rate="$(arg baud_rate)"/>
 </robot>

Commit message: feat(dynamixel_node): fix hardware interface export, add servo mocking, normalize angles, harden set_mode
- Call base class SystemInterface::on_init(params) so the framework
  populates joint_state/command interface maps from the URDF
- Add mock_servo_ids hardware parameter to simulate missing servos
  in software (skips bus scan, torque, read/write for listed IDs)
- Add normalizeAngle ([-pi,pi]) for read path and normalizeAnglePositive
  ([0,2pi)) for write path to handle Dynamixel encoder wraparound
- Disable torque before changing operating mode (Dynamixel protocol
  requirement; fixes "Motor torque status mismatch" on restart)
- Skip non-finite command values in write() to prevent out_of_range
  crash on the first cycle before controllers set commands
- Increase baud rate from 57600 to 1000000 in xacro
- Wire mock_servo_ids through xacro and launch file

File: src/arm_moveit_config/config/arm.ros2_control.xacro (robot description, xacro)
@@ -1,5 +1,5 @@
 <?xml version="1.0"?>
 <robot xmlns:xacro="http://www.ros.org/wiki/xacro">
-    <xacro:macro name="arm_ros2_control" params="name initial_positions_file use_mock_hardware:=false hardware_plugin:=dynamixel_node/DynamixelServos">
+    <xacro:macro name="arm_ros2_control" params="name initial_positions_file use_mock_hardware:=false hardware_plugin:=dynamixel_node/DynamixelServos mock_servo_ids:=''">
         <xacro:property name="initial_positions" value="${xacro.load_yaml(initial_positions_file)['initial_positions']}"/>
         <ros2_control name="${name}" type="system">
@@ -11,5 +11,6 @@
                   <plugin>${hardware_plugin}</plugin>
                   <param name="device">/dev/ttyUSB0</param>
-                  <param name="baud_rate">57600</param>
+                  <param name="baud_rate">1000000</param>
+                  <param name="mock_servo_ids">${mock_servo_ids}</param>
                 </xacro:unless>
             </hardware>

File: src/arm_moveit_config/config/arm.urdf.xacro (robot description, xacro)
@@ -4,8 +4,9 @@
     <xacro:arg name="use_mock_hardware" default="true" />
     <xacro:arg name="hardware_plugin" default="dynamixel_node/DynamixelServos" />
+    <xacro:arg name="mock_servo_ids" default="" />
     <!-- Import arm urdf file -->
     <xacro:include filename="$(find arm_moveit_config)/src/moveit/arm.urdf" />
     <!-- Import control_xacro -->
     <xacro:include filename="arm.ros2_control.xacro" />
-    <xacro:arm_ros2_control name="DynamixelServos" initial_positions_file="$(arg initial_positions_file)" use_mock_hardware="$(arg use_mock_hardware)" hardware_plugin="$(arg hardware_plugin)"/>
+    <xacro:arm_ros2_control name="DynamixelServos" initial_positions_file="$(arg initial_positions_file)" use_mock_hardware="$(arg use_mock_hardware)" hardware_plugin="$(arg hardware_plugin)" mock_servo_ids="$(arg mock_servo_ids)"/>
 </robot>
